File: the NFT.kicad_pcb (KiCad board)
At the start: 4 copper layers, 131.5 x 98.7 mm, 95 parts, among them J1 USB_C_Receptacle_USB2.0_16P, J10 Conn_01x06, J11 Conn_01x12, J2 Conn_01x02, J3 Conn_01x02, J4 Screw_Terminal_01x03, J5 Screw_Terminal_01x03, J6 Screw_Terminal_01x03, J7 Screw_Terminal_01x03, J8 Screw_Terminal_01x03, J9 Screw_Terminal_01x03, K2 JQC-3FF-012-1Z, K3 JQC-3FF-012-1Z, K4 JQC-3FF-012-1Z, K5 JQC-3FF-012-1Z, K6 JQC-3FF-012-1Z, K7 JQC-3FF-012-1Z, Q1 S8050, Q2 S8050, Q3 S8050, Q4 S8050, Q5 S8050, Q6 S8050, Q7 S8050, Q8 S8050, SW4 SW_SPST, SW5 SW_SPST, SW6 SW_SPST, SW7 SW_SPST, SW8 SW_SPST, SW9 SW_SPST, U1 LM2596S-5, U2 ESP32-WROOM-32, U3 AMS1117-3.3, U4 CH340C, U5 ADS1115IDGS, U6 BME280, U7 MB85RC256VPNF-G-AMERE2

Commit message: Add files via upload
Parts:
- removed C2: 1uF, Capacitor_SMD:C_0805_2012Metric
- removed C3: 100nF, Capacitor_SMD:C_0805_2012Metric
- removed C4: 10uF, Capacitor_SMD:C_0805_2012Metric
- removed C7: 22uF, Capacitor_SMD:C_Elec_5x5.4
- removed D1: 1N5822, Diode_SMD:D_SMC
- removed DC1: DC-C033D-5.5A-2.0, EasyEDA:DC-IN-TH_DC-C033D-5.5A-2.5
- removed R1: 1kΩ, Resistor_SMD:R_0805_2012Metric
- removed R17: 4.7kΩ, Resistor_SMD:R_0805_2012Metric
- removed R34: 22, Resistor_SMD:R_0805_2012Metric
- removed R9: 2kΩ, Resistor_SMD:R_0805_2012Metric
- removed S2: B3U-1000P, Button_Switch_SMD:SW_SPST_B3U-1000P
- removed U2: ESP32-WROOM-32, RF_Module:ESP32-S3-WROOM-1
- added C13: 100nf, Capacitor_SMD:C_0805_2012Metric, F.Cu at (136.1, 71.2)
- added C14: 100nf, Capacitor_SMD:C_0805_2012Metric, F.Cu at (128.8, 78.5)
- added C15: 100nf, Capacitor_SMD:C_0805_2012Metric, F.Cu at (136.5, 63.8)
- added C16: 10uf, Capacitor_SMD:C_0805_2012Metric, F.Cu at (136.4, 66.0)
- added C17: 22uF 10v, Capacitor_SMD:CP_Elec_5x5.4, F.Cu at (202.0, 107.0)
- added C18: 100nf, Capacitor_SMD:C_0805_2012Metric, F.Cu at (112.2, 84.5)
- added C21: 1000uf, Capacitor_SMD:CP_Elec_10x10.5, F.Cu at (209.2, 124.5)
- added C26: 100nf, Capacitor_SMD:C_0805_2012Metric, F.Cu at (124.0, 90.2)
- added CR2: SK34A-LTP, SK34A-LTP:SMADO-214AC_MCC, F.Cu at (212.5, 139.2)
- added G***: LOGO, LOGO, F.Cu at (197.8, 90.0)
- added JP11: SolderJumper_3_Bridged12, Jumper:SolderJumper-3_P1.3mm_Bridged12_Pad1.0x1.5mm, F.Cu at (108.5, 80.5)
- added R2: 1kΩ, Resistor_SMD:R_0805_2012Metric, F.Cu at (119.8, 78.5)
- added R33: 10k, Resistor_SMD:R_0805_2012Metric, F.Cu at (136.1, 73.5)
- added R35: 22, Resistor_SMD:R_0805_2012Metric, F.Cu at (131.8, 77.7)
- added R38: 10k, Resistor_SMD:R_0805_2012Metric, F.Cu at (128.8, 76.2)
- added R4: 2kΩ, Resistor_SMD:R_0805_2012Metric, F.Cu at (115.8, 78.5)
- added R47: 10k, Resistor_SMD:R_0805_2012Metric, F.Cu at (104.9, 84.5)
- added R49: 10k, Resistor_SMD:R_0805_2012Metric, F.Cu at (108.6, 84.5)
- added S1: B3U-1000P, B3U-1000P:SW_B3U-1000P, F.Cu at (138.0, 79.2)
- added U8: ESP32-S3-WROOM-1(N16R8), lcsc_footprints:C2913202_WIRELM-SMD_ESP32-S3-WROOM-1, F.Cu at (152.5, 67.9)
- J11: value Conn_01x12 -> DC-005 2.0mm; footprint Connector_PinHeader_2.54mm:PinHeader_1x12_P2.54mm_Vertical -> lcsc_footprints:C84007_DC-IN-TH_DC-005C-20A
- J3: value Conn_01x02 -> Conn_01x15; footprint Connector_PinHeader_2.54mm:PinHeader_1x02_P2.54mm_Vertical -> Connector_PinHeader_2.54mm:PinHeader_1x15_P2.54mm_Vertical
- S3: footprint Button_Switch_SMD:SW_SPST_B3U-1000P -> B3U-1000P:SW_B3U-1000P
- moved J11 84.6 mm to (214.5, 145.5), turned to 90 degrees
- moved J10 9.59 mm to (219.0, 104.5)
- moved I2C1 7.59 mm to (219.0, 121.1)
- moved J3 7.58 mm to (219.5, 60.7), turned to 0 degrees
- moved D9 7.29 mm to (181.5, 96.2)
- moved vout1 6.50 mm to (215.5, 132.5), turned to 90 degrees
- moved S3 3.20 mm to (134.8, 79.2)
- moved SW5 0.51 mm to (123.7, 142.2)
- moved U5 0.16 mm to (118.6, 89.2)
Connections:
- Conn_01x04 pad 2: Net-(Conn_01x04-Pin_2) -> IO17
- I2C1 pad 3: IO22/SCL -> IO42/SCL
- J10 pad 3: IO23/MOSI -> IO41/MOSI
- J11 pad 1: SCS/CMD -> Net-(CR2-Pad2)
- J11 pad 2: SCK/CLK -> GND
- J11 pad 3: SWP/SD3 -> GND
- J3 pad 1: Net-(J3-Pin_1) -> IO1
- J3 pad 2: Net-(J3-Pin_2) -> IO2
- R10 pad 2: IO26 -> IO40
- R12 pad 2: IO22/SCL -> IO42/SCL
- R13 pad 2: IO27 -> IO39
- R16 pad 2: IO22 -> IO42/SCL
- R19 pad 2: IO34 -> IO36
- S3 pad 1: Net-(C3-Pad1) -> GND
- S3 pad 2: GND -> Net-(R35-Pad2)
- U5 pad 1: GND -> Net-(JP11-C)
- U5 pad 10: IO22 -> IO42/SCL
- U5 pad 2: unconnected-(U5-ALERT/RDY-Pad2) -> Net-(U5-ALERT/RDY)
- U5 pad 9: IO21 -> IO21/SDA
- U6 pad 4: IO22/SCL -> IO42/SCL
- U7 pad 6: IO22/SCL -> IO42/SCL
Routing:
- net IO42/SCL: track 0.00 -> 217.1 mm, vias 0 -> 4
- net IO22/SCL: track 135.4 -> 0.00 mm, vias 2 -> 0
- net IO34: track 107.8 -> 0.00 mm, vias 3 -> 0
- net IO36: track 0.00 -> 106.2 mm, vias 0 -> 3
- net IO39: track 0.00 -> 94.2 mm, vias 0 -> 2
- net IO41/MOSI: track 0.00 -> 92.2 mm, vias 0 -> 2
- net SCS/CMD: track 91.9 -> 0.00 mm, vias 1 -> 0
- net IO32: track 87.2 -> 0.00 mm, vias 3 -> 0
- net IO21/SDA: track 137.4 -> 223.1 mm, vias 3 -> 6
- net IO7: track 0.00 -> 84.3 mm, vias 0 -> 3
- net IO40: track 0.00 -> 82.6 mm, vias 0 -> 4
- net IO6: track 0.00 -> 81.9 mm, vias 0 -> 3
- net IO25: track 81.9 -> 0.00 mm, vias 4 -> 0
- net IO8: track 0.00 -> 81.8 mm, vias 0 -> 3
- net SWP/SD3: track 81.7 -> 0.00 mm, vias 2 -> 0
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Other:
- board size 131.5 x 98.7 mm -> 131.9 x 99 mm
- board text added: "12V"
- board text added: "12V ONLY"
- board text added: "3.3"
- board text added: "3.3V"
- board text added: "5V"
- board text added: "AIN 1"
- board text added: "AIN 2"
- board text added: "CS"
- board text added: "EC ANALOG"
- board text added: "ECHO"
- board text added: "GND"
- board text added: "IO1"
- board text added: "IO10"
- board text added: "IO11"
- board text added: "IO12"
- board text added: "IO13"
- board text added: "IO14"
- board text added: "IO15"
- board text added: "IO16"
- board text added: "IO2"
- board text added: "IO20"
- board text added: "IO35"
- board text added: "IO36"
- board text added: "IO37"
- board text added: "IO38"
- board text added: "IO39"
- board text added: "IO40"
- board text added: "IO6"
- board text added: "IO7"
- board text added: "IO8"
- board text added: "IO9"
- board text added: "MISO"
- board text added: "MOSI"
- board text added: "PH ANALOG"
- board text added: "PLUG V"
- board text added: "SCK"
- board text added: "SCL"
- board text added: "SDA"
- board text added: "TRIG"
