File: the NFT.kicad_sch (KiCad schematic)
At the start: 94 parts, among them J1 USB_C_Receptacle_USB2.0_16P, J10 Conn_01x06, J11 Conn_01x12, J2 Conn_01x02, J3 Conn_01x02, J4 Screw_Terminal_01x03, J5 Screw_Terminal_01x03, J6 Screw_Terminal_01x03, J7 Screw_Terminal_01x03, J8 Screw_Terminal_01x03, J9 Screw_Terminal_01x03, K2 JQC-3FF-012-1Z, K3 JQC-3FF-012-1Z, K4 JQC-3FF-012-1Z, K5 JQC-3FF-012-1Z, K6 JQC-3FF-012-1Z, K7 JQC-3FF-012-1Z, Q1 S8050, Q2 S8050, Q3 S8050, Q4 S8050, Q5 S8050, Q6 S8050, Q7 S8050, Q8 S8050, SW4 SW_SPST, SW5 SW_SPST, SW6 SW_SPST, SW7 SW_SPST, SW8 SW_SPST, SW9 SW_SPST, U1 LM2596S-5, U2 ESP32-WROOM-32, U3 AMS1117-3.3, U4 CH340C, U5 ADS1115IDGS, U6 BME280, U7 MB85RC256VPNF-G-AMERE2

Commit message: Add files via upload
Parts:
- removed C2: 1uF, Capacitor_SMD:C_0805_2012Metric, symbol Device:C
- removed C3: 100nF, Capacitor_SMD:C_0805_2012Metric, symbol Device:C
- removed C4: 10uF, Capacitor_SMD:C_0805_2012Metric, symbol Device:C
- removed C7: 22uF, Capacitor_SMD:C_Elec_5x5.4, symbol Device:C
- removed DC1: DC-C033D-5.5A-2.0, EasyEDA:DC-IN-TH_DC-C033D-5.5A-2.5, symbol EasyEDA:DC-C033D-5.5A-2.0
- removed J11: Conn_01x12, Connector_PinHeader_2.54mm:PinHeader_1x12_P2.54mm_Vertical, symbol Connector_Generic:Conn_01x12
- removed J3: Conn_01x02, Connector_PinHeader_2.54mm:PinHeader_1x02_P2.54mm_Vertical, symbol Connector_Generic:Conn_01x02
- removed R16, R17: 4.7kΩ, Resistor_SMD:R_0805_2012Metric, symbol Device:R
- removed R34: 22, Resistor_SMD:R_0805_2012Metric, symbol Device:R
- removed R4, R7: 10kΩ, Resistor_SMD:R_0805_2012Metric, symbol Device:R
- removed R9: 2kΩ, Resistor_SMD:R_0805_2012Metric, symbol Device:R
- removed S2: B3U-1000P, Button_Switch_SMD:SW_SPST_B3U-1000P, symbol B3U-1000P:B3U-1000P
- removed U2: ESP32-WROOM-32, RF_Module:ESP32-S3-WROOM-1, symbol RF_Module:ESP32-WROOM-32
- added C13, C14, C15, C18, C26: 100nf, Capacitor_SMD:C_0805_2012Metric, symbol Device:C
- added C16: 10uf, Capacitor_SMD:C_0805_2012Metric, symbol Device:C
- added C17: 22uF 10v, Capacitor_SMD:CP_Elec_5x5.4, symbol Device:C_Polarized
- added CR2: SK34A-LTP, SK34A-LTP:SMADO-214AC_MCC, symbol SK34A-LTP:SK34A-LTP
- added J11: DC-005 2.0mm, lcsc_footprints:C84007_DC-IN-TH_DC-005C-20A, symbol lcsc_imported:DC-005_2_0mm
- added J3: Conn_01x15, Connector_PinHeader_2.54mm:PinHeader_1x15_P2.54mm_Vertical, symbol Connector_Generic:Conn_01x15
- added JP11: SolderJumper_3_Bridged12, Jumper:SolderJumper-3_P1.3mm_Bridged12_Pad1.0x1.5mm, symbol Jumper:SolderJumper_3_Bridged12
- added R2: 1kΩ, Resistor_SMD:R_0805_2012Metric, symbol Device:R
- added R33, R38, R47, R49: 10k, Resistor_SMD:R_0805_2012Metric, symbol Device:R
- added R35: 22, Resistor_SMD:R_0805_2012Metric, symbol Device:R
- added S1: B3U-1000P, B3U-1000P:SW_B3U-1000P, symbol B3U-1000P:B3U-1000P
- added U8: ESP32-S3-WROOM-1(N16R8), lcsc_footprints:C2913202_WIRELM-SMD_ESP32-S3-WROOM-1, symbol lcsc_imported:ESP32-S3-WROOM-1(N16R8)
- C5: LCSC part (none) -> C3345
- F3: LCSC part (none) -> C70138
- J1: LCSC part (none) -> C720628
- S3: footprint Button_Switch_SMD:SW_SPST_B3U-1000P -> B3U-1000P:SW_B3U-1000P
Connections:
- net IO21 is gone; now on net IO21/SDA: U5.9 (SDA)
- net IO22/SCL is gone; now on net IO42/SCL: I2C1.3 (Pin_3), R12.2, U6.4 (SCK), U7.6 (SCL)
- net +12v: now also CR2.1
- net +3v3: now also C15.2, C16.1, C17.1, C18.2, C26.2, J3.14 (Pin_14), JP11.1 (A), R33.1, R38.1, R47.1, U8.2 (3V3)
- net C-Q1: now also C14.2, R35.1, R38.2, U8.3 (EN)
- net C-Q2: now also C13.2, R33.2, S1.2, U8.27 (IO0)
- net GND: now also S3.1, C13.1, C14.1, C15.1, C16.2, C17.2, C18.1, C26.1, J11.2, J11.3, J3.15 (Pin_15), R49.2, S1.1, U8.1 (GND), U8.40 (GND), U8.41 (GND); no longer S3.2, U5.1 (ADDR)
- net IO12: now also U8.20 (IO12)
- net IO13: now also U8.21 (IO13)
- net IO14: now also U8.22 (IO14)
- net IO15: now also J3.13 (Pin_13), U8.8 (IO15)
- net IO16: now also J3.12 (Pin_12), U8.9 (IO16)
- net IO17: now also R2.1
- net IO18/SCK: now also U8.11 (IO18)
- net IO19/MISO: now also U8.13 (IO19)
- net IO2: now also J3.2 (Pin_2), U8.38 (IO2)
- net IO21/SDA: now also U8.23 (IO21)
- net IO35: now also U8.28 (IO35)
- net IO4: now also U8.4 (IO4)
- net IO5/CS: now also U8.5 (IO5)
- net RX-ESP32: now also U8.36 (RXD0)
- net TX-ESP32: now also U8.37 (TXD0)
- net at U5.2 (ALERT/RDY): now also R47.2
- net IO22 renamed IO42/SCL
- net IO42/SCL: now also U8.35 (IO42)
- net IO23/MOSI renamed IO41/MOSI
- net IO41/MOSI: now also U8.34 (IO41)
- net IO26 renamed IO40
- net IO40: now also U8.33 (IO40)
- net IO27 renamed IO39
- net IO39: now also U8.32 (IO39)
- net IO34 renamed IO36
- net IO36: now also U8.29 (IO36)
- new net: R2.2, U8.10 (IO17)
- new net: CR2.2, J11.1
- new net: JP11.2 (C), U5.1 (ADDR)
- new net: JP11.3 (B), R49.1
- new net: R35.2, S3.2
- new net IO1: J3.1 (Pin_1), U8.39 (IO1)
- new net IO10: J3.7 (Pin_7), U8.18 (IO10)
- new net IO11: J3.8 (Pin_8), U8.19 (IO11)
- new net IO20: J3.11 (Pin_11), U8.14 (IO20)
- new net IO37: J3.9 (Pin_9), U8.30 (IO37)
- new net IO38: J3.10 (Pin_10), U8.31 (IO38)
- new net IO6: J3.3 (Pin_3), U8.6 (IO6)
- new net IO7: J3.4 (Pin_4), U8.7 (IO7)
- new net IO8: J3.5 (Pin_5), U8.12 (IO8)
- new net IO9: J3.6 (Pin_6), U8.17 (IO9)
- no-connect marks 8 -> 18
Other:
- note added: "I2C: 0x48"
- moved on the sheet: C12, C5, C9, D4, I2C1, J10, J2, R11, R12, U7, vout1
